File: CP2104_UART-USB_micro_B.sch (KiCad schematic (older format))
At the start: 8 parts

Commit message: semi schematiced
Parts:
- C5, C6: renamed from C?; footprint (none) -> Capacitor_SMD:C_0805_2012Metric_Pad1.18x1.45mm_HandSolder
- J2: renamed from J?; footprint (none) -> Connector_USB:USB_Micro-B_GCT_USB3076-30-A
- R1, R2, R3: renamed from R?; footprint (none) -> Resistor_SMD:R_0805_2012Metric_Pad1.20x1.40mm_HandSolder
- gave numbers to parts that had none: 2
Connections:
- net GND: now also J2.5 (GND), J2.6 (Shield)
- net at U4.3 (D+): now also U3.4; no longer U3.6
- net at U4.4 (D-): now also U3.6; no longer U3.4
- net at J2.2 (D-): now also U3.1; no longer U3.3
- net at J2.3 (D+): now also U3.3; no longer U3.1
Changed lines of the file:
@@
 P 3450 3100
 AR Path="/606D9181" Ref="J?"  Part="1"
-AR Path="/606D7E2A/606D9181" Ref="J?"  Part="1"
-F 0 "J?" H 3507 3567 50  0000 C CNN
+AR Path="/606D7E2A/606D9181" Ref="J2"  Part="1"
+F 0 "J2" H 3507 3567 50  0000 C CNN
 F 1 "USB_B_Micro" H 3507 3476 50  0000 C CNN
-F 2 "" H 3600 3050 50  0001 C CNN
+F 2 "Connector_USB:USB_Micro-B_GCT_USB3076-30-A" H 3600 3050 50  0001 C CNN
 F 3 "~" H 3600 3050 50  0001 C CNN
 	1    3450 3100
@@
 P 5100 2750
 AR Path="/606D9187" Ref="R?"  Part="1"
-AR Path="/606D7E2A/606D9187" Ref="R?"  Part="1"
-F 0 "R?" V 4893 2750 50  0000 C CNN
+AR Path="/606D7E2A/606D9187" Ref="R1"  Part="1"
+F 0 "R1" V 4893 2750 50  0000 C CNN
 F 1 "24K" V 4984 2750 50  0000 C CNN
-F 2 "" V 5030 2750 50  0001 C CNN
+F 2 "Resistor_SMD:R_0805_2012Metric_Pad1.20x1.40mm_HandSolder" V 5030 2750 50  0001 C CNN
 F 3 "~" H 5100 2750 50  0001 C CNN
 	1    5100 2750
@@
 P 5300 2550
 AR Path="/606D918D" Ref="R?"  Part="1"
-AR Path="/606D7E2A/606D918D" Ref="R?"  Part="1"
-F 0 "R?" H 5230 2504 50  0000 R CNN
+AR Path="/606D7E2A/606D918D" Ref="R2"  Part="1"
+F 0 "R2" H 5230 2504 50  0000 R CNN
 F 1 "47K" H 5230 2595 50  0000 R CNN
-F 2 "" V 5230 2550 50  0001 C CNN
+F 2 "Resistor_SMD:R_0805_2012Metric_Pad1.20x1.40mm_HandSolder" V 5230 2550 50  0001 C CNN
 F 3 "~" H 5300 2550 50  0001 C CNN
 	1    5300 2550
@@
 P 7500 3650
 AR Path="/606D9193" Ref="R?"  Part="1"
-AR Path="/606D7E2A/606D9193" Ref="R?"  Part="1"
-F 0 "R?" V 7707 3650 50  0000 C CNN
+AR Path="/606D7E2A/606D9193" Ref="R3"  Part="1"
+F 0 "R3" V 7707 3650 50  0000 C CNN
 F 1 "1K" V 7616 3650 50  0000 C CNN
-F 2 "" V 7430 3650 50  0001 C CNN
+F 2 "Resistor_SMD:R_0805_2012Metric_Pad1.20x1.40mm_HandSolder" V 7430 3650 50  0001 C CNN
 F 3 "~" H 7500 3650 50  0001 C CNN
 	1    7500 3650
@@
 $EndComp
 $Comp
-L Device:C C?
+L Device:C C5
 U 1 1 606D9435
 P 5400 4050
-F 0 "C?" H 5515 4096 50  0000 L CNN
+F 0 "C5" H 5515 4096 50  0000 L CNN
 F 1 "1uF" H 5515 4005 50  0000 L CNN
-F 2 "" H 5438 3900 50  0001 C CNN
+F 2 "Capacitor_SMD:C_0805_2012Metric_Pad1.18x1.45mm_HandSolder" H 5438 3900 50  0001 C CNN
 F 3 "~" H 5400 4050 50  0001 C CNN
 	1    5400 4050
@@
 $EndComp
 $Comp
-L Device:C C?
+L Device:C C6
 U 1 1 606D9B62
 P 6750 2200
-F 0 "C?" V 6498 2200 50  0000 C CNN
+F 0 "C6" V 6498 2200 50  0000 C CNN
 F 1 "C" V 6589 2200 50  0000 C CNN
-F 2 "" H 6788 2050 50  0001 C CNN
+F 2 "Capacitor_SMD:C_0805_2012Metric_Pad1.18x1.45mm_HandSolder" H 6788 2050 50  0001 C CNN
 F 3 "~" H 6750 2200 50  0001 C CNN
 	1    6750 2200
@@
 	7200 2750 7050 2750
 $Comp
-L power:+3V3 #PWR?
+L power:+3V3 #PWR0116
 U 1 1 606DAECA
 P 6350 2150
-F 0 "#PWR?" H 6350 2000 50  0001 C CNN
+F 0 "#PWR0116" H 6350 2000 50  0001 C CNN
 F 1 "+3V3" H 6365 2323 50  0000 C CNN
 F 2 "" H 6350 2150 50  0001 C CNN
@@
 $EndComp
 $Comp
-L power:GND #PWR?
+L power:GND #PWR0117
 U 1 1 606DB330
 P 6450 4300
-F 0 "#PWR?" H 6450 4050 50  0001 C CNN
+F 0 "#PWR0117" H 6450 4050 50  0001 C CNN
 F 1 "GND" H 6455 4127 50  0000 C CNN
 F 2 "" H 6450 4300 50  0001 C CNN
@@
 $EndComp
 $Comp
-L power:+5V #PWR?
+L power:+5V #PWR0118
 U 1 1 606DC218
 P 4900 2750
-F 0 "#PWR?" H 4900 2600 50  0001 C CNN
+F 0 "#PWR0118" H 4900 2600 50  0001 C CNN
 F 1 "+5V" H 4915 2923 50  0000 C CNN
 F 2 "" H 4900 2750 50  0001 C CNN
@@
 $EndComp
 $Comp
-L Power_Protection:WE-TVS-82400102 U?
+L Power_Protection:WE-TVS-82400102 U3
 U 1 1 606DCFFE
 P 4500 3150
-F 0 "U?" H 4500 3475 50  0000 C CNN
-F 1 "WE-TVS-82400102" H 4500 3384 50  0000 C CNN
+F 0 "U3" H 4500 2835 50  0000 C CNN
+F 1 "WE-TVS-82400102" H 4500 2926 50  0000 C CNN
 F 2 "Package_TO_SOT_SMD:SOT-23-6" H 4500 2950 50  0001 C CNN
 F 3 "https://katalog.we-online.de/pbs/datasheet/82400102.pdf" H 4500 2900 50  0001 C CNN
 	1    4500 3150
-	1    0    0    -1
-$EndComp
-$Comp
-L power:GND #PWR?
+	1    0    0    1
+$EndComp
+$Comp
+L power:GND #PWR0119
 U 1 1 606E0670
 P 4200 3150
-F 0 "#PWR?" H 4200 2900 50  0001 C CNN
+F 0 "#PWR0119" H 4200 2900 50  0001 C CNN
 F 1 "GND" V 4205 3022 50  0000 R CNN
 F 2 "" H 4200 3150 50  0001 C CNN
@@
 	5300 2750 5650 2750
 $Comp
-L power:GND #PWR?
+L power:GND #PWR0120
 U 1 1 606F3109
 P 5300 2400
-F 0 "#PWR?" H 5300 2150 50  0001 C CNN
+F 0 "#PWR0120" H 5300 2150 50  0001 C CNN
 F 1 "GND" H 5305 2227 50  0000 C CNN
 F 2 "" H 5300 2400 50  0001 C CNN
@@
 P 6350 3150
 AR Path="/606D917B" Ref="U?"  Part="1"
-AR Path="/606D7E2A/606D917B" Ref="U?"  Part="1"
-F 0 "U?" H 6600 2150 50  0000 C CNN
+AR Path="/606D7E2A/606D917B" Ref="U4"  Part="1"
+F 0 "U4" H 6600 2150 50  0000 C CNN
 F 1 "CP2104" H 6700 2050 50  0000 C CNN
 F 2 "Package_DFN_QFN:QFN-24-1EP_4x4mm_P0.5mm_EP2.6x2.6mm" H 6500 2200 50  0001 L CNN
@@
 	6550 2200 6350 2200
 $Comp
-L power:GND #PWR?
+L power:GND #PWR0121
 U 1 1 606F709C
 P 6900 2200
-F 0 "#PWR?" H 6900 1950 50  0001 C CNN
+F 0 "#PWR0121" H 6900 1950 50  0001 C CNN
 F 1 "GND" V 6905 2072 50  0000 R CNN
 F 2 "" H 6900 2200 50  0001 C CNN
@@
 	5400 3850 5400 3900
 $Comp
-L power:GND #PWR?
+L power:GND #PWR0122
 U 1 1 606F94F4
 P 5400 4300
-F 0 "#PWR?" H 5400 4050 50  0001 C CNN
+F 0 "#PWR0122" H 5400 4050 50  0001 C CNN
 F 1 "GND" H 5405 4127 50  0000 C CNN
 F 2 "" H 5400 4300 50  0001 C CNN
@@
 	7050 3650 7350 3650
 $Comp
-L power:+3V3 #PWR?
+L power:+3V3 #PWR0123
 U 1 1 606FB65D
 P 7800 3650
-F 0 "#PWR?" H 7800 3500 50  0001 C CNN
+F 0 "#PWR0123" H 7800 3500 50  0001 C CNN
 F 1 "+3V3" H 7815 3823 50  0000 C CNN
 F 2 "" H 7800 3650 50  0001 C CNN
@@
 Text HLabel 7200 3350 2    50   Output ~ 0
 RTS
+$Comp
+L power:GND #PWR?
+U 1 1 607E90F4
+P 3450 3550
+F 0 "#PWR?" H 3450 3300 50  0001 C CNN
+F 1 "GND" H 3455 3377 50  0000 C CNN
+F 2 "" H 3450 3550 50  0001 C CNN
+F 3 "" H 3450 3550 50  0001 C CNN
+	1    3450 3550
+	1    0    0    -1
+$EndComp
+Wire Wire Line
+	3350 3500 3350 3550
+Wire Wire Line
+	3350 3550 3450 3550
+Wire Wire Line
+	3450 3550 3450 3500
+Connection ~ 3450 3550
 $EndSCHEMATC
