File: ESP32_S2_strip.kicad_pcb (KiCad board)
At the start: 2 copper layers, 64.2 x 35 mm, 38 parts, among them J1 Barrel_Jack_Switch, J2 USB_B_Micro, J3 Conn_01x02_Male, J4 Conn_01x02_Male, Q1 MBT3904DW1, U1 LM1117-3.3, U2 ESP32-S2-WROVER, U3 WE-TVS-82400102, U4 CP2104

Commit message: Rev 1
Parts:
- added G***: LOGO, Andrew_van_dam_logo:Andrew_van_dam_logo_12mm, F.Cu at (79.5, -5.21)
- moved 4_PIN 7.61 mm to (122.2, -18.8), turned to 180 degrees
- moved I2C 2.61 mm to (118.5, -24.8)
- moved C7 1.75 mm to (84.0, -9.50)
- moved 3_PIN 1.25 mm to (122.2, -9.00)
- moved U2 1.16 mm to (97.2, -20.0)
- renumbered 3_PIN1 to 3_PIN, 4_PIN1 to 4_PIN, FLASH1 to FLASH, I2C1 to I2C, RESET1 to RESET, J2 to USB
Routing:
- net GND: track 52.2 -> 117.3 mm, vias 7 -> 12
- net +3V3: track 32.9 -> 85.7 mm, vias 2 -> 4
- net WS281x: track 0.00 -> 47.3 mm
- net /ESP32_USB_auto_reset/GPIO0: track 12.5 -> 50.6 mm
- net DATA: track 0.00 -> 36.2 mm, vias 0 -> 2
- net CLK: track 0.00 -> 35.7 mm, vias 0 -> 4
- net /ESP32_USB_auto_reset/CHIP_PU: track 9.19 -> 38.0 mm
- net ADC1: track 0.00 -> 23.6 mm
- net Net-(R8-Pad2): track 0.00 -> 23.4 mm, vias 0 -> 2
- net I2C_CLK: track 0.00 -> 23.4 mm
- net I2C_DATA: track 0.00 -> 20.9 mm
- net ADC0: track 0.00 -> 19.4 mm
- net ESP32_RX: track 0.00 -> 18.5 mm, vias 0 -> 2
- net Net-(R9-Pad2): track 0.00 -> 18.3 mm, vias 0 -> 2
- net ESP32_TX: track 0.00 -> 15.7 mm, vias 0 -> 2
- added copper zone on B.Cu, net GND
- added copper zone on B.Cu, net VCC
Other:
- board text added: "0"
- board text added: "1"
- board text added: "3V3"
- board text added: "C"
- board text added: "D"
- board text added: "DOUT"
- board text added: "GND"
- board text added: "PB_0"
- board text added: "PB_1"
- board text added: "VIN"
