File: ESP32_S2_strip.sch (KiCad schematic (older format))
At the start: 9 parts

Commit message: Preliminary schematic capture
Parts:
- added 3_PIN, ADC_1: Conn_01x03_Male, symbol Connector:Conn_01x03_Male
- added 4_PIN: Conn_01x04_Male, Connector_PinHeader_2.54mm:PinHeader_1x04_P2.54mm_Horizontal, symbol Connector:Conn_01x04_Male
- added ADC_0: Conn_01x03_Male, Connector_PinHeader_2.54mm:PinHeader_1x03_P2.54mm_Horizontal, symbol Connector:Conn_01x03_Male
- J?: footprint (none) -> Connector_BarrelJack:BarrelJack_CUI_PJ-102AH_Horizontal
Connections:
- net +3V3: now also ADC_0.1 (Pin_1), ADC_1.1 (Pin_1)
- net GND: now also 3_PIN.3 (Pin_3), 4_PIN.4 (Pin_4), ADC_0.3 (Pin_3), ADC_1.3 (Pin_3)
- net VCC: now also 3_PIN.1 (Pin_1), 4_PIN.1 (Pin_1)
- net I2C_CLK: now reaches U?.12 (IO09)
- net I2C_DATA: now reaches U?.13 (IO10)
- net WS281x: now reaches U?.21 (IO18)
- net WS281x: now also 3_PIN.2 (Pin_2)
- net DATA: now reaches U?.29 (IO35)
- net DATA: now also 4_PIN.3 (Pin_3)
- net CLK: now reaches U?.30 (IO36)
- net CLK: now also 4_PIN.2 (Pin_2)
- net ADC0: now reaches U?.4 (IO01)
- net ADC0: now also ADC_0.2 (Pin_2)
- net ADC1: now reaches U?.5 (IO02)
- net ADC1: now also ADC_1.2 (Pin_2)
Changed lines of the file:
@@
 F 0 "J?" H 2907 4367 50  0000 C CNN
 F 1 "Barrel_Jack_Switch" H 2907 4276 50  0000 C CNN
-F 2 "" H 2900 4010 50  0001 C CNN
+F 2 "Connector_BarrelJack:BarrelJack_CUI_PJ-102AH_Horizontal" H 2900 4010 50  0001 C CNN
 F 3 "~" H 2900 4010 50  0001 C CNN
 	1    2850 4050
@@
 Wire Wire Line
 	7200 2350 7300 2350
+Text GLabel 5550 2550 0    50   Input ~ 0
+ADC0
+Text GLabel 5550 2650 0    50   Input ~ 0
+ADC1
+Wire Wire Line
+	5550 2550 5700 2550
+Wire Wire Line
+	5700 2550 5700 2250
+Wire Wire Line
+	5700 2250 6000 2250
+Wire Wire Line
+	5550 2650 5750 2650
+Wire Wire Line
+	5750 2650 5750 2350
+Wire Wire Line
+	5750 2350 6000 2350
+Text GLabel 5850 3950 0    50   Input ~ 0
+WS281x
+$Comp
+L Connector:Conn_01x03_Male ADC_0
+U 1 1 6072E9E1
+P 3700 5850
+F 0 "ADC_0" H 3672 5874 50  0000 R CNN
+F 1 "Conn_01x03_Male" H 3672 5783 50  0000 R CNN
+F 2 "Connector_PinHeader_2.54mm:PinHeader_1x03_P2.54mm_Horizontal" H 3700 5850 50  0001 C CNN
+F 3 "~" H 3700 5850 50  0001 C CNN
+	1    3700 5850
+	-1   0    0    -1
+$EndComp
+$Comp
+L Connector:Conn_01x03_Male ADC_1
+U 1 1 6072FA8F
+P 3700 6550
+F 0 "ADC_1" H 3672 6574 50  0000 R CNN
+F 1 "Conn_01x03_Male" H 3672 6483 50  0000 R CNN
+F 2 "" H 3700 6550 50  0001 C CNN
+F 3 "~" H 3700 6550 50  0001 C CNN
+	1    3700 6550
+	-1   0    0    -1
+$EndComp
+$Comp
+L Connector:Conn_01x03_Male 3_PIN
+U 1 1 60730473
+P 6000 5550
+F 0 "3_PIN" H 5972 5574 50  0000 R CNN
+F 1 "Conn_01x03_Male" H 5972 5483 50  0000 R CNN
+F 2 "" H 6000 5550 50  0001 C CNN
+F 3 "~" H 6000 5550 50  0001 C CNN
+	1    6000 5550
+	-1   0    0    -1
+$EndComp
+Text GLabel 7500 3050 2    50   Input ~ 0
+CLK
+Text GLabel 7500 3150 2    50   Input ~ 0
+DATA
+Text GLabel 5700 5550 0    50   Input ~ 0
+WS281x
+Text GLabel 3450 5850 0    50   Input ~ 0
+ADC0
+Text GLabel 3450 6550 0    50   Input ~ 0
+ADC1
+$Comp
+L power:+3V3 #PWR?
+U 1 1 607314B3
+P 3450 5750
+F 0 "#PWR?" H 3450 5600 50  0001 C CNN
+F 1 "+3V3" H 3465 5923 50  0000 C CNN
+F 2 "" H 3450 5750 50  0001 C CNN
+F 3 "" H 3450 5750 50  0001 C CNN
+	1    3450 5750
+	1    0    0    -1
+$EndComp
+$Comp
+L power:+3V3 #PWR?
+U 1 1 607320E2
+P 3450 6450
+F 0 "#PWR?" H 3450 6300 50  0001 C CNN
+F 1 "+3V3" H 3465 6623 50  0000 C CNN
+F 2 "" H 3450 6450 50  0001 C CNN
+F 3 "" H 3450 6450 50  0001 C CNN
+	1    3450 6450
+	1    0    0    -1
+$EndComp
+$Comp
+L power:GND #PWR?
+U 1 1 60733531
+P 3450 5950
+F 0 "#PWR?" H 3450 5700 50  0001 C CNN
+F 1 "GND" H 3455 5777 50  0000 C CNN
+F 2 "" H 3450 5950 50  0001 C CNN
+F 3 "" H 3450 5950 50  0001 C CNN
+	1    3450 5950
+	1    0    0    -1
+$EndComp
+$Comp
+L power:GND #PWR?
+U 1 1 60733CB6
+P 3450 6650
+F 0 "#PWR?" H 3450 6400 50  0001 C CNN
+F 1 "GND" H 3455 6477 50  0000 C CNN
+F 2 "" H 3450 6650 50  0001 C CNN
+F 3 "" H 3450 6650 50  0001 C CNN
+	1    3450 6650
+	1    0    0    -1
+$EndComp
+Wire Wire Line
+	3450 6450 3500 6450
+Wire Wire Line
+	3500 6550 3450 6550
+Wire Wire Line
+	3450 6650 3500 6650
+Wire Wire Line
+	3500 5950 3450 5950
+Wire Wire Line
+	3450 5850 3500 5850
+Wire Wire Line
+	3500 5750 3450 5750
+Wire Wire Line
+	5700 5550 5800 5550
+$Comp
+L Connector:Conn_01x04_Male 4_PIN
+U 1 1 6073861C
+P 6000 6250
+F 0 "4_PIN" H 5972 6224 50  0000 R CNN
+F 1 "Conn_01x04_Male" H 5972 6133 50  0000 R CNN
+F 2 "Connector_PinHeader_2.54mm:PinHeader_1x04_P2.54mm_Horizontal" H 6000 6250 50  0001 C CNN
+F 3 "~" H 6000 6250 50  0001 C CNN
+	1    6000 6250
+	-1   0    0    -1
+$EndComp
+Text GLabel 5650 6250 0    50   Input ~ 0
+CLK
+Text GLabel 5650 6350 0    50   Input ~ 0
+DATA
+$Comp
+L power:GND #PWR?
+U 1 1 6073AA8B
+P 5750 5650
+F 0 "#PWR?" H 5750 5400 50  0001 C CNN
+F 1 "GND" H 5755 5477 50  0000 C CNN
+F 2 "" H 5750 5650 50  0001 C CNN
+F 3 "" H 5750 5650 50  0001 C CNN
+	1    5750 5650
+	1    0    0    -1
+$EndComp
+$Comp
+L power:GND #PWR?
+U 1 1 6073B16D
+P 5750 6450
+F 0 "#PWR?" H 5750 6200 50  0001 C CNN
+F 1 "GND" H 5755 6277 50  0000 C CNN
+F 2 "" H 5750 6450 50  0001 C CNN
+F 3 "" H 5750 6450 50  0001 C CNN
+	1    5750 6450
+	1    0    0    -1
+$EndComp
+$Comp
+L power:VCC #PWR?
+U 1 1 6073B839
+P 5750 6150
+F 0 "#PWR?" H 5750 6000 50  0001 C CNN
+F 1 "VCC" H 5765 6323 50  0000 C CNN
+F 2 "" H 5750 6150 50  0001 C CNN
+F 3 "" H 5750 6150 50  0001 C CNN
+	1    5750 6150
+	1    0    0    -1
+$EndComp
+Wire Wire Line
+	5650 6350 5800 6350
+Wire Wire Line
+	5800 6450 5750 6450
+Wire Wire Line
+	5650 6250 5800 6250
+Wire Wire Line
+	5800 6150 5750 6150
+Wire Wire Line
+	5750 5650 5800 5650
+$Comp
+L power:VCC #PWR?
+U 1 1 607402A5
+P 5750 5450
+F 0 "#PWR?" H 5750 5300 50  0001 C CNN
+F 1 "VCC" H 5765 5623 50  0000 C CNN
+F 2 "" H 5750 5450 50  0001 C CNN
+F 3 "" H 5750 5450 50  0001 C CNN
+	1    5750 5450
+	1    0    0    -1
+$EndComp
+Wire Wire Line
+	5750 5450 5800 5450
+Wire Wire Line
+	5850 3950 6000 3950
+Wire Wire Line
+	7200 3050 7500 3050
+Wire Wire Line
+	7500 3150 7200 3150
+Text GLabel 5800 3050 0    50   Input ~ 0
+I2C_CLK
+Text GLabel 5800 3150 0    50   Input ~ 0
+I2C_DATA
+Wire Wire Line
+	5800 3050 6000 3050
+Wire Wire Line
+	6000 3150 5800 3150
 $EndSCHEMATC

Commit message: semi schematiced
Parts:
- removed U?: AMS1117-3.3, Package_TO_SOT_SMD:SOT-223-3_TabPin2, symbol Regulator_Linear:AMS1117-3.3
- added DC_IN1: Screw_Terminal_01x02, TerminalBlock_4Ucon:TerminalBlock_4Ucon_1x02_P3.50mm_Horizontal, symbol Connector:Screw_Terminal_01x02
- added I2C1: Conn_01x04_Male, Connector_PinHeader_2.54mm:PinHeader_1x04_P2.54mm_Vertical, symbol Connector:Conn_01x04_Male
- added J3, J4: Conn_01x02_Male, Connector_PinHeader_2.54mm:PinHeader_1x02_P2.54mm_Vertical, symbol Connector:Conn_01x02_Male
- added R8, R9: 1K, Resistor_SMD:R_0805_2012Metric_Pad1.20x1.40mm_HandSolder, symbol Device:R
- added SW_0, SW_1: SW_Push, Button_Switch_SMD:SW_Push_1P1T_NO_CK_KMR2, symbol Switch:SW_Push
- added U1: LM1117-3.3, Package_TO_SOT_SMD:SOT-223-3_TabPin2, symbol Regulator_Linear:LM1117-3.3
- 3_PIN1: renamed from 3_PIN; footprint (none) -> Connector_PinHeader_2.54mm:PinHeader_1x03_P2.54mm_Vertical
- 4_PIN1: renamed from 4_PIN; footprint Connector_PinHeader_2.54mm:PinHeader_1x04_P2.54mm_Horizontal -> Connector_PinHeader_2.54mm:PinHeader_1x04_P2.54mm_Vertical
- ADC_0: footprint Connector_PinHeader_2.54mm:PinHeader_1x03_P2.54mm_Horizontal -> Connector_PinHeader_2.54mm:PinHeader_1x03_P2.54mm_Vertical
- ADC_1: footprint (none) -> Connector_PinHeader_2.54mm:PinHeader_1x03_P2.54mm_Vertical
- C1, C2, C3, C4: renamed from C?; footprint (none) -> Capacitor_SMD:C_0805_2012Metric_Pad1.18x1.45mm_HandSolder
- FB1, FB2: renamed from FB?; footprint (none) -> Resistor_SMD:R_0603_1608Metric_Pad0.98x0.95mm_HandSolder; Digikey (none) -> 283-MFBW1V1608-101-RCT-ND
- J1: renamed from J?; Digikey (none) -> CP-102AH-ND
- U2: renamed from U?; Digikey (none) -> 1965-ESP32-S2-WROVERCT-ND
Connections:
- net +3V3: now also I2C1.1 (Pin_1)
- net GND: now also J1.2, DC_IN1.2 (Pin_2), I2C1.4 (Pin_4), J3.2 (Pin_2), J4.2 (Pin_2), SW_0.2, SW_1.2, U1.1 (GND)
- net I2C_CLK: now also I2C1.2 (Pin_2)
- net I2C_DATA: now also I2C1.3 (Pin_3)
- net VCC: now also DC_IN1.1 (Pin_1)
- net at U2.27 (IO33): now also R9.2
- net at U2.28 (IO34): now also R8.2
- net at FB2.2: now also U1.2 (VO)
- net at C1.1, FB1.1: now also U1.3 (VI)
- new net: J3.1 (Pin_1), R8.1, SW_0.1
- new net: J4.1 (Pin_1), R9.1, SW_1.1

Commit message: Rev 1
Changed lines of the file:
@@
+	1    0    0    -1
+$EndComp
+$Comp
+L Andrew_van_dam_logo:LOGO #G1
+U 1 1 606FC633
+P 9400 6000
+F 0 "#G1" H 9400 5801 60  0001 C CNN
+F 1 "LOGO" H 9400 6199 60  0001 C CNN
+F 2 "Andrew_van_dam_logo:Andrew_van_dam_logo_12mm" H 9400 6000 50  0001 C CNN
+F 3 "" H 9400 6000 50  0001 C CNN
+	1    9400 6000
 	1    0    0    -1
 $EndComp
